File: hard/GPduino-T/GPduino-T.brd (EAGLE design)
At the start: 68.6 x 48.3 mm, 56 parts, among them CN1 EH-3-POWER, CN2 MINI-USB-UX60A-MB-5ST, CN3 EH-4, CN4 EH-4, CN5 EH-2, CN6 EH-2, CN7 , Q1 IRLML8244, Q2 IRLML8244, SW1 SKRPACE010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

Commit message: rev.2基板
Parts:
- added R21, R22: 100, SparkFun:0603-RES
- added VR1: 10k, lipoyang_discrete:EVM3Y
- C3: value 220uF -> 0.1uF; device rcl:UD-6,3X7,7_NICHICON -> resistor:C1608
- C4: value 0.1uF -> 220uF; device resistor:C1608 -> rcl:UD-6,3X7,7_NICHICON
- CN2: value MINI-USB-UX60A-MB-5ST -> EH-4; device lipoyang_mechanical:UX60A-MB-5ST -> lipoyang_mechanical:EH-4
- CN3: value EH-4 -> MINI-USB-UX60A-MB-5ST; device lipoyang_mechanical:EH-4 -> lipoyang_mechanical:UX60A-MB-5ST
- R10, R11: value 10K -> 100
- R12, R13: value 100 -> 10K
- R3: value 10K -> 1.5K
- R4: value 10K -> 680
- R6, R7: value 150 -> 10K
- R8, R9: value 100 -> 150
- U1: value NCP1117 -> OKL-T/3-W12N; device lipoyang_ic:SOT223 -> lipoyang_ic:OKL-T/X-WXXN
- U4: device esp32:ESP-WROOM-32 -> lipoyang_rf:ESP-WROOM-32
- moved CN2 62.9 mm to (66.7, 25.4), turned to 270 degrees
- moved CN3 62.9 mm to (6.35, 7.62), turned to 0 degrees
- moved C3 44.6 mm to (5.71, 14.6), turned to 180 degrees
- moved C4 34.4 mm to (36.8, 29.2), turned to 0 degrees
- moved R7 31.1 mm to (9.21, 17.8), turned to 90 degrees
- moved R9 30.6 mm to (28.9, 41.9), turned to 270 degrees
- moved R8 27.4 mm to (31.8, 35.9), turned to 0 degrees
- moved R4 23.5 mm to (43.5, 29.5)
- moved R6 22.0 mm to (25.1, 14.9)
- moved R5 18.9 mm to (27.9, 20.6)
- moved R3 18.9 mm to (43.5, 31.4), turned to 180 degrees
- moved R12 16.2 mm to (45.4, 8.26), turned to 90 degrees
- moved R17 13.6 mm to (38.1, 8.26), turned to 90 degrees
- moved R18 13.6 mm to (40.6, 8.26), turned to 90 degrees
- moved R13 11.4 mm to (21.6, 8.89), turned to 0 degrees
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- renumbered CN7 to JP4
Connections:
- new net N$33: C12.2, VR1.2
- new net N$35: R3.1, R4.2
- new net N$36: R3.2, U1.6
- net +3V3: now also C4.+, R6.2, R7.2, U1.4@1, U1.5; no longer C3.+, R3.2, R4.2, U1.2
- net A01: now also CN2.4; no longer CN3.4
- net A02: now also CN2.3; no longer CN3.3
- net GND: now also C3.2, C4.-, CN3.5, R12.1, R13.1, R4.1, U1.3, U1.3@2, U1.3@3, U1.7, VR1.3; no longer C3.-, C4.2, CN2.5, R10.1, R11.1
- net IR_LED: now also R11.2; no longer R9.2
- net IR_LED_SINK: now also R14.2; no longer R12.2
- net LED0: now also R15.1; no longer R13.1
- net LED1: now also R16.1; no longer R14.1
- net LED2: now also R17.1; no longer R15.1
- net LED3: now also R18.1; no longer R16.1
- net LED4: now also R19.1; no longer R17.1
- net LED5: now also R20.1; no longer R18.1
- net LED6: now also R21.1; no longer R19.1
- net LED7: now also R22.1; no longer R20.1
- net N$12: now also R22.2; no longer R20.2
- net N$13: now also CN3.2; no longer CN2.2
- net N$14: now also CN3.3; no longer CN2.3
- net N$16: now also R21.2; no longer R19.2
- net N$17: now also R20.2; no longer R18.2
- net N$18: now also R19.2; no longer R17.2
- net N$19: now also R18.2; no longer R16.2
- net N$20: now also R17.2; no longer R15.2
- net N$21: now also R16.2; no longer R14.2
- net N$22: now also R15.2; no longer R13.2
- net N$23: now also R8.1; no longer R6.1
- net N$24: now also R9.1; no longer R7.1
- net N$26: now also R8.2; no longer R6.2
- net N$27: now also R9.2; no longer R7.2
- net N$3: now also R10.1, R12.2; no longer R10.2, R8.1
- net N$5: now also CN2.1; no longer CN3.1
- net N$6: now also CN2.2; no longer CN3.2
- net N$7: now also R11.1, R13.2; no longer R11.2, R9.1
- net N$8: now also R14.1; no longer R12.1
- net RESET: now also R7.1; no longer R5.1
- net SCL: now also R5.1; no longer R3.1
- net SDA: now also R6.1; no longer R4.1
- net SOLENOID: now also R10.2; no longer R8.2
- net SOUND: now also VR1.1; no longer C12.2
- net VBUS: now also C3.1, CN3.1; no longer C4.1, CN2.1
- net V_BATT: now also U1.2, U1.2@2, U1.2@3; no longer U1.3
Routing:
- net SOUND: track 18.4 -> 13.9 mm
- net +3V3: track 183.1 -> 178.7 mm, vias 28 -> 1
- net N$33: track 0.00 -> 4.19 mm
- net V_BATT: track 82.2 -> 78.7 mm
- net N$36: track 0.00 -> 3.33 mm
- net N$35: track 0.00 -> 1.91 mm
- net GND: track 0.00 -> 1.46 mm, vias 63 -> 59
- added copper zone on layer 1, net N$34
- removed copper zone on layer 16, net +3V3
